File: pcb/main/AFF314MODKEEB.kicad_pcb (KiCad board)
At the start: 2 copper layers, 206.5 x 70.5 mm, 103 parts, among them SW1 SW_Push_45deg, SW10 SW_Push_45deg, SW11 SW_Push_45deg, SW12 SW_Push_45deg, SW13 SW_Push_45deg, SW14 SW_Push_45deg, SW15 SW_Push_45deg, SW16 SW_Push_45deg, SW17 SW_Push_45deg, SW18 SW_Push_45deg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

Commit message: update pcb & add firmware
Parts:
- moved SW49 0.50 mm to (41.0, 79.9)
Routing:
- net unconnected-(SW49-Pad2): track 25.8 -> 36.9 mm, vias 1 -> 2
- net unconnected-(SW49-Pad3): track 21.8 -> 21.3 mm
