File: pcb/main/AFF314MODKEEB.kicad_sch (KiCad schematic)
At the start: 102 parts, among them SW1 SW_Push_45deg, SW10 SW_Push_45deg, SW11 SW_Push_45deg, SW12 SW_Push_45deg, SW13 SW_Push_45deg, SW14 SW_Push_45deg, SW15 SW_Push_45deg, SW16 SW_Push_45deg, SW17 SW_Push_45deg, SW18 SW_Push_45deg, SW19 SW_Push_45deg, SW2 SW_Push_45deg, SW20 SW_Push_45deg, SW21 SW_Push_45deg, SW22 SW_Push_45deg, SW23 SW_Push_45deg, SW24 SW_Push_45deg, SW25 SW_Push_45deg, SW26 SW_Push_45deg, SW27 SW_Push_45deg, SW28 SW_Push_45deg, SW29 SW_Push_45deg, SW3 SW_Push_45deg, SW30 SW_Push_45deg, SW31 SW_Push_45deg, SW32 SW_Push_45deg, SW33 SW_Push_45deg, SW34 SW_Push_45deg, SW35 SW_Push_45deg, SW36 SW_Push_45deg, SW37 SW_Push_45deg, SW38 SW_Push_45deg, SW39 SW_Push_45deg, SW4 SW_Push_45deg, SW40 SW_Push_45deg, SW41 SW_Push_45deg, SW42 SW_Push_45deg, SW43 SW_Push_45deg, SW44 SW_Push_45deg, SW45 SW_Push_45deg, SW46 SW_Push_45deg, SW47 SW_Push_45deg, SW48 SW_Push_45deg, SW49 SK12D07VG3_C431547, SW5 SW_Push_45deg, SW6 SW_Push_45deg, SW7 SW_Push_45deg, SW8 SW_Push_45deg, SW9 SW_Push_45deg, U6 Nice_Nano_V2

Commit message: update pcb & add firmware
Parts:
- added BT1: Battery, symbol Device:Battery
Connections:
- net COL 0: now also U6.9 (6)
- net COL 1: now also U6.10 (7)
- net COL 10: now also U6.14 (16)
- net COL 11: now also U6.13 (10)
- net COL 12: now also U3.3, U6.25 (1)
- net COL 13: now also U3.2, U6.26 (2)
- net COL 14: now also U3.1, U6.27 (7)
- net COL 2: now also U6.11 (8)
- net COL 3: now also U6.12 (9)
- net COL 4: now also U6.20 (21)
- net COL 5: now also U6.19 (20)
- net COL 6: now also U6.18 (19)
- net COL 7: now also U6.17 (18)
- net COL 8: now also U6.16 (15)
- net COL 9: now also U6.15 (14)
- net GND: now also SW49.2, U6.3 (GND)
- net ROW 0: now also U2.5, U6.1
- net ROW 1: now also U2.4, U6.2 (0)
- net ROW 2: now also U6.5 (2)
- net ROW 3: now also U2.3, U6.6 (3)
- net ROW 4: now also U2.2, U6.7 (4)
- net ROW 5: now also U2.1, U6.8 (5)
- net at SW49.1: now also BT1.1 (+)
- net BAT: now reaches U6.24 (B+)
- net BAT: now also BT1.2 (-)
Other:
- note added: "bottom 6pin"
- note added: "left 8pin"
- note added: "mcu"
- note added: "powerswitch"
- note added: "right 8pin"
- note added: "top 6pin"
- moved on the sheet: SW49
