File: pcb/right/module_right.kicad_pcb (KiCad board)
At the start: 2 copper layers, 54.4 x 88.5 mm, 23 parts, among them SW1 SW_Push_45deg, SW2 SW_Push_45deg, SW3 SW_Push_45deg, SW4 SW_Push_45deg, SW5 SW_Push_45deg, SW6 SW_Push_45deg, SW7 SW_Push_45deg, SW8 SW_Push_45deg, SW9 SW_Push_45deg

Commit message: update pcb & add firmware
Parts:
- removed ENC1: RotaryEncoder_Switch, AFFElib:RotaryEncoder_Alps_EC11E-Switch_Vertical_H20mm
- added SW10: SW_Push_45deg, AFFElib:choc_16, F.Cu at (135.5, 55.8)
- moved DR1 8.49 mm to (131.8, 52.5)
Routing:
- net COL 14: track 82.8 -> 109.6 mm
- net COL 13: track 105.8 -> 124.6 mm
- net COL 12: track 90.9 -> 109.6 mm
- net Net-(DR1-A): track 5.39 -> 21.7 mm
- net ROW 4: track 33.4 -> 32.2 mm
- net GND: track 0.02 -> 0.00 mm, vias 1 -> 0
- net B: vias 1 -> 0
- net A: vias 1 -> 0
