File: pcb/right/module_right.kicad_sch (KiCad schematic)
At the start: 23 parts, among them SW1 SW_Push_45deg, SW2 SW_Push_45deg, SW3 SW_Push_45deg, SW4 SW_Push_45deg, SW5 SW_Push_45deg, SW6 SW_Push_45deg, SW7 SW_Push_45deg, SW8 SW_Push_45deg, SW9 SW_Push_45deg

Commit message: update pcb & add firmware
Parts:
- removed ENC1: RotaryEncoder_Switch, AFFElib:RotaryEncoder_Alps_EC11E-Switch_Vertical_H20mm, symbol Device:RotaryEncoder_Switch
- removed U1: (no value), symbol ScottoKeebs:magnetic11_male
- added SW10: SW_Push_45deg, AFFElib:choc_16, symbol Switch:SW_Push_45deg
Connections:
- net A is gone; now on net COL 13: U3.5
- net GND is gone; now on net COL 12: U3.4
- net ROW 4 is gone; now on net ROW 3: D1.1 (K), D2.1 (K), DR1.1 (K)
- net COL 12: no longer U3.6
- net COL 13: no longer U2.1
- net COL 14: now also U3.6, SW10.1; no longer U2.2
- net ROW 2: now also D3.1 (K), D4.1 (K), D5.1 (K)
- net ROW 3: no longer D3.1 (K), D4.1 (K), D5.1 (K)
- net at DR1.2 (A): now also SW10.2
- net B: no longer names the net of U3.3
Other:
- note added: "bottom 6pin"
- note added: "top 6pin"
- moved on the sheet: D1, D2, D3, D4, D5, D6, D7, D8, D9, DR1, SW1, SW2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
