File: pcb/top2/module_top2.kicad_sch (KiCad schematic)
At the start: 50 parts, among them SW1 SW_Push_45deg, SW10 SW_Push_45deg, SW11 SW_Push_45deg, SW12 SW_Push_45deg, SW13 SW_Push_45deg, SW14 SW_Push_45deg, SW15 SW_Push_45deg, SW16 SW_Push_45deg, SW17 SW_Push_45deg, SW18 SW_Push_45deg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

Commit message: update pcb & add firmware
Other:
- note added: "left 8pin"
- note added: "right 8pin"
Changed lines of the file:
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@@
 	(generator_version "10.0")
 	(paper "A4")
+	(text "left 8pin"
+		(exclude_from_sim no)
+		(at 68.326 130.302 0)
+		(effects
+			(font
+				(size 1.27 1.27)
+			)
+		)
+	)
+	(text "right 8pin"
+		(exclude_from_sim no)
+		(at 111.76 130.048 0)
+		(effects
+			(font
+				(size 1.27 1.27)
+			)
+		)
+	)
 	(junction
 		(at 133.35 92.71)
